File: pcb_files/AI4R-PIHAT/AI4R-PIHAT.kicad_pcb (KiCad board)
At the start: 2 copper layers, 65 x 56 mm, 15 parts, among them J1 Conn_02x20_Odd_Even, J2 Conn_01x04, J3 Conn_01x04, J4 Conn_01x04, J5 Conn_01x04, J6 Conn_02x10_Odd_Even, J7 Conn_01x03, J8 Conn_01x03, J9 Conn_01x02, U1 815

Commit message: fix gerber errors
Connections:
- U1 pad VCC: VCC -> 3.3V
Routing:
- net 3.3V: track 132.8 -> 161.4 mm, vias 1 -> 0
- net VCC: track 84.9 -> 85.5 mm
Other:
- board text added: "V1.1 Aug 2024"
- board text removed: "V1.0 June 2024"
